File: hardware/bredtoob.sch (EAGLE design)
At the start: 55 parts

Commit message: v02
Swap half the noval tube sockets for b7g sockets so we support almost all miniature tubes (compactrons notwithstanding)

Radius the corners of the board

Reduce rails to 40 pins to match common header strips

Add bus headers beside each breadboard to reduce mess if you need to wire between the two
Parts:
- removed J10, J11, J12, J13, J14, J15, J16, J17, J18, J19, J20, J21, J22, J23, J24, J3, J4, J5, J6, J7, J8, J9: (no value), SparkFun-Connectors:CONN_16
- added J43, J44, J45, J46, J47, J48: (no value), SparkFun-Connectors:CONN_40
- J1, J2: device SparkFun-Connectors:CONN_16 -> SparkFun-Connectors:CONN_10NO_SILK_PTH_FEMALE
- J26, J28, J30, J31, J33, J35: device SparkFun-Connectors:CONN_09 -> SparkFun-Connectors:CONN_07NO_SILK
- U$11, U$2, U$4, U$6, U$7, U$9: value 9PINMINI -> 7PINMINI; device Toob:9PINMINI -> Toob:7PINMINI
Connections:
- removed net N$105: J35.1, U$11.P$9
- removed net N$16: J26.9, U$2.P$1
- removed net N$24: J26.1, U$2.P$9
- removed net N$34: J28.9, U$4.P$1
- removed net N$42: J28.1, U$4.P$9
- removed net N$52: J30.9, U$6.P$1
- removed net N$60: J30.1, U$6.P$9
- removed net N$61: J31.9, U$7.P$1
- removed net N$69: J31.1, U$7.P$9
- removed net N$79: J33.9, U$9.P$1
- removed net N$87: J33.1, U$9.P$9
- removed net N$97: J35.9, U$11.P$1
- new net A: J1.1, J2.1
- new net B: J1.2, J2.2
- new net C: J1.3, J2.3
- new net D: J1.4, J2.4
- new net E: J1.5, J2.5
- new net F: J1.6, J2.6
- new net G: J1.7, J2.7
- new net H: J1.8, J2.8
- new net I: J1.9, J2.9
- new net J: J1.10, J2.10
- net GND: now also J44.1, J44.10, J44.11, J44.12, J44.13, J44.14, J44.15, J44.16, J44.17, J44.18, J44.19, J44.2, J44.20, J44.21, J44.22, J44.23, J44.24, J44.25, J44.26, J44.27, J44.28, J44.29, J44.3, J44.30, J44.31, J44.32, J44.33, J44.34, J44.35, J44.36, J44.37, J44.38, J44.39, J44.4, J44.40, J44.5, J44.6, J44.7, J44.8, J44.9, J47.1, J47.10, J47.11, J47.12, J47.13, J47.14, J47.15, J47.16, J47.17, J47.18, J47.19, J47.2, J47.20, J47.21, J47.22, J47.23, J47.24, J47.25, J47.26, J47.27, J47.28, J47.29, J47.3, J47.30, J47.31, J47.32, J47.33, J47.34, J47.35, J47.36, J47.37, J47.38, J47.39, J47.4, J47.40, J47.5, J47.6, J47.7, J47.8, J47.9; no longer J1.1, J1.10, J1.11, J1.12, J1.13, J1.14, J1.15, J1.16, J1.2, J1.3, J1.4, J1.5, J1.6, J1.7, J1.8, J1.9, J13.1, J13.10, J13.11, J13.12, J13.13, J13.14, J13.15, J13.16, J13.2, J13.3, J13.4, J13.5, J13.6, J13.7, J13.8, J13.9, J14.1, J14.10, J14.11, J14.12, J14.13, J14.14, J14.15, J14.16, J14.2, J14.3, J14.4, J14.5, J14.6, J14.7, J14.8, J14.9, J15.1, J15.10, J15.11, J15.12, J15.13, J15.14, J15.15, J15.16, J15.2, J15.3, J15.4, J15.5, J15.6, J15.7, J15.8, J15.9, J16.1, J16.10, J16.11, J16.12, J16.13, J16.14, J16.15, J16.16, J16.2, J16.3, J16.4, J16.5, J16.6, J16.7, J16.8, J16.9, J2.1, J2.10, J2.11, J2.12, J2.13, J2.14, J2.15, J2.16, J2.2, J2.3, J2.4, J2.5, J2.6, J2.7, J2.8, J2.9, J3.1, J3.10, J3.11, J3.12, J3.13, J3.14, J3.15, J3.16, J3.2, J3.3, J3.4, J3.5, J3.6, J3.7, J3.8, J3.9, J4.1, J4.10, J4.11, J4.12, J4.13, J4.14, J4.15, J4.16, J4.2, J4.3, J4.4, J4.5, J4.6, J4.7, J4.8, J4.9
- net N$1: now also J43.1, J43.10, J43.11, J43.12, J43.13, J43.14, J43.15, J43.16, J43.17, J43.18, J43.19, J43.2, J43.20, J43.21, J43.22, J43.23, J43.24, J43.25, J43.26, J43.27, J43.28, J43.29, J43.3, J43.30, J43.31, J43.32, J43.33, J43.34, J43.35, J43.36, J43.37, J43.38, J43.39, J43.4, J43.40, J43.5, J43.6, J43.7, J43.8, J43.9; no longer J10.1, J10.10, J10.11, J10.12, J10.13, J10.14, J10.15, J10.16, J10.2, J10.3, J10.4, J10.5, J10.6, J10.7, J10.8, J10.9, J11.1, J11.10, J11.11, J11.12, J11.13, J11.14, J11.15, J11.16, J11.2, J11.3, J11.4, J11.5, J11.6, J11.7, J11.8, J11.9, J12.1, J12.10, J12.11, J12.12, J12.13, J12.14, J12.15, J12.16, J12.2, J12.3, J12.4, J12.5, J12.6, J12.7, J12.8, J12.9, J9.1, J9.10, J9.11, J9.12, J9.13, J9.14, J9.15, J9.16, J9.2, J9.3, J9.4, J9.5, J9.6, J9.7, J9.8, J9.9
- net N$100: now also J31.5, U$11.P$3; no longer J35.6, U$11.P$4
- net N$101: now also J31.4, U$11.P$4; no longer J35.5, U$11.P$5
- net N$102: now also J31.3, U$11.P$5; no longer J35.4, U$11.P$6
- net N$103: now also J31.2, U$11.P$6; no longer J35.3, U$11.P$7
- net N$104: now also J31.1, U$11.P$7; no longer J35.2, U$11.P$8
- net N$17: now also J26.7, U$2.P$1; no longer J26.8, U$2.P$2
- net N$18: now also J26.6, U$2.P$2; no longer J26.7, U$2.P$3
- net N$19: now also J26.5, U$2.P$3; no longer J26.6, U$2.P$4
- net N$2: now also J45.1, J45.10, J45.11, J45.12, J45.13, J45.14, J45.15, J45.16, J45.17, J45.18, J45.19, J45.2, J45.20, J45.21, J45.22, J45.23, J45.24, J45.25, J45.26, J45.27, J45.28, J45.29, J45.3, J45.30, J45.31, J45.32, J45.33, J45.34, J45.35, J45.36, J45.37, J45.38, J45.39, J45.4, J45.40, J45.5, J45.6, J45.7, J45.8, J45.9; no longer J17.1, J17.10, J17.11, J17.12, J17.13, J17.14, J17.15, J17.16, J17.2, J17.3, J17.4, J17.5, J17.6, J17.7, J17.8, J17.9, J18.1, J18.10, J18.11, J18.12, J18.13, J18.14, J18.15, J18.16, J18.2, J18.3, J18.4, J18.5, J18.6, J18.7, J18.8, J18.9, J19.1, J19.10, J19.11, J19.12, J19.13, J19.14, J19.15, J19.16, J19.2, J19.3, J19.4, J19.5, J19.6, J19.7, J19.8, J19.9, J20.1, J20.10, J20.11, J20.12, J20.13, J20.14, J20.15, J20.16, J20.2, J20.3, J20.4, J20.5, J20.6, J20.7, J20.8, J20.9
- net N$20: now also J26.4, U$2.P$4; no longer J26.5, U$2.P$5
- net N$21: now also J26.3, U$2.P$5; no longer J26.4, U$2.P$6
- net N$22: now also J26.2, U$2.P$6; no longer J26.3, U$2.P$7
- net N$23: now also J26.1, U$2.P$7; no longer J26.2, U$2.P$8
- net N$3: now also J46.1, J46.10, J46.11, J46.12, J46.13, J46.14, J46.15, J46.16, J46.17, J46.18, J46.19, J46.2, J46.20, J46.21, J46.22, J46.23, J46.24, J46.25, J46.26, J46.27, J46.28, J46.29, J46.3, J46.30, J46.31, J46.32, J46.33, J46.34, J46.35, J46.36, J46.37, J46.38, J46.39, J46.4, J46.40, J46.5, J46.6, J46.7, J46.8, J46.9; no longer J21.1, J21.10, J21.11, J21.12, J21.13, J21.14, J21.15, J21.16, J21.2, J21.3, J21.4, J21.5, J21.6, J21.7, J21.8, J21.9, J22.1, J22.10, J22.11, J22.12, J22.13, J22.14, J22.15, J22.16, J22.2, J22.3, J22.4, J22.5, J22.6, J22.7, J22.8, J22.9, J23.1, J23.10, J23.11, J23.12, J23.13, J23.14, J23.15, J23.16, J23.2, J23.3, J23.4, J23.5, J23.6, J23.7, J23.8, J23.9, J24.1, J24.10, J24.11, J24.12, J24.13, J24.14, J24.15, J24.16, J24.2, J24.3, J24.4, J24.5, J24.6, J24.7, J24.8, J24.9
- net N$35: now also J28.7, U$4.P$1; no longer J28.8, U$4.P$2
- net N$36: now also J28.6, U$4.P$2; no longer J28.7, U$4.P$3
- net N$37: now also J28.5, U$4.P$3; no longer J28.6, U$4.P$4
- net N$38: now also J28.4, U$4.P$4; no longer J28.5, U$4.P$5
- net N$39: now also J28.3, U$4.P$5; no longer J28.4, U$4.P$6
- net N$4: now also J48.1, J48.10, J48.11, J48.12, J48.13, J48.14, J48.15, J48.16, J48.17, J48.18, J48.19, J48.2, J48.20, J48.21, J48.22, J48.23, J48.24, J48.25, J48.26, J48.27, J48.28, J48.29, J48.3, J48.30, J48.31, J48.32, J48.33, J48.34, J48.35, J48.36, J48.37, J48.38, J48.39, J48.4, J48.40, J48.5, J48.6, J48.7, J48.8, J48.9; no longer J5.1, J5.10, J5.11, J5.12, J5.13, J5.14, J5.15, J5.16, J5.2, J5.3, J5.4, J5.5, J5.6, J5.7, J5.8, J5.9, J6.1, J6.10, J6.11, J6.12, J6.13, J6.14, J6.15, J6.16, J6.2, J6.3, J6.4, J6.5, J6.6, J6.7, J6.8, J6.9, J7.1, J7.10, J7.11, J7.12, J7.13, J7.14, J7.15, J7.16, J7.2, J7.3, J7.4, J7.5, J7.6, J7.7, J7.8, J7.9, J8.1, J8.10, J8.11, J8.12, J8.13, J8.14, J8.15, J8.16, J8.2, J8.3, J8.4, J8.5, J8.6, J8.7, J8.8, J8.9
- net N$40: now also J28.2, U$4.P$6; no longer J28.3, U$4.P$7
- net N$41: now also J28.1, U$4.P$7; no longer J28.2, U$4.P$8
- net N$53: now also J30.7, U$6.P$1; no longer J30.8, U$6.P$2
- net N$54: now also J30.6, U$6.P$2; no longer J30.7, U$6.P$3
- net N$55: now also J30.5, U$6.P$3; no longer J30.6, U$6.P$4
- net N$56: now also J30.4, U$6.P$4; no longer J30.5, U$6.P$5
- net N$57: now also J30.3, U$6.P$5; no longer J30.4, U$6.P$6
- net N$58: now also J30.2, U$6.P$6; no longer J30.3, U$6.P$7
- net N$59: now also J30.1, U$6.P$7; no longer J30.2, U$6.P$8
- net N$62: now also J35.7, U$7.P$1; no longer J31.8, U$7.P$2
- net N$63: now also J35.6, U$7.P$2; no longer J31.7, U$7.P$3
- net N$64: now also J35.5, U$7.P$3; no longer J31.6, U$7.P$4
- net N$65: now also J35.4, U$7.P$4; no longer J31.5, U$7.P$5
- net N$66: now also J35.3, U$7.P$5; no longer J31.4, U$7.P$6
- net N$67: now also J35.2, U$7.P$6; no longer J31.3, U$7.P$7
- net N$68: now also J35.1, U$7.P$7; no longer J31.2, U$7.P$8
- net N$80: now also J33.7, U$9.P$1; no longer J33.8, U$9.P$2
- net N$81: now also J33.6, U$9.P$2; no longer J33.7, U$9.P$3
- net N$82: now also J33.5, U$9.P$3; no longer J33.6, U$9.P$4
- net N$83: now also J33.4, U$9.P$4; no longer J33.5, U$9.P$5
- net N$84: now also J33.3, U$9.P$5; no longer J33.4, U$9.P$6
- net N$85: now also J33.2, U$9.P$6; no longer J33.3, U$9.P$7
- net N$86: now also J33.1, U$9.P$7; no longer J33.2, U$9.P$8
- net N$98: now also J31.7, U$11.P$1; no longer J35.8, U$11.P$2
- net N$99: now also J31.6, U$11.P$2; no longer J35.7, U$11.P$3
Other:
- moved on the sheet: J39, J42

Commit message: v03
Glad I waited for parts to come in for testing before ordering v02

- Replace banana jack headers with binding posts
- Widen Pin Receptacle headers to accept Mill-Max 0312-0-15-80-34-80-10-0
- Revise Silkscreen Labels
- Add OSHW Logo
Parts:
- removed J37, J38, J39, J40, J41, J42: (no value), SparkFun-Connectors:BANANA_CONN
- added J3, J4, J5, J6, J7, J8: BINDING_POST, SparkFun-Connectors:BINDING_POST
Connections:
- net GND: now also J3.P$1, J4.P$1; no longer J37.1, J38.1
- net N$1: now also J5.P$1; no longer J39.1
- net N$2: now also J6.P$1; no longer J40.1
- net N$3: now also J7.P$1; no longer J42.1
- net N$4: now also J8.P$1; no longer J41.1
Changed lines of the file:
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@@
 <part name="GND1" library="SparkFun-PowerSymbols" deviceset="GND" device=""/>
 <part name="GND2" library="SparkFun-PowerSymbols" deviceset="GND" device=""/>
-<part name="J37" library="SparkFun-Connectors" deviceset="BANANA_CONN" device=""/>
-<part name="J38" library="SparkFun-Connectors" deviceset="BANANA_CONN" device=""/>
-<part name="J39" library="SparkFun-Connectors" deviceset="BANANA_CONN" device=""/>
-<part name="J40" library="SparkFun-Connectors" deviceset="BANANA_CONN" device=""/>
-<part name="J41" library="SparkFun-Connectors" deviceset="BANANA_CONN" device=""/>
-<part name="J42" library="SparkFun-Connectors" deviceset="BANANA_CONN" device=""/>
 <part name="GND3" library="SparkFun-PowerSymbols" deviceset="GND" device=""/>
 <part name="J26" library="SparkFun-Connectors" deviceset="CONN_07" device="NO_SILK"/>
@@
 <part name="J1" library="SparkFun-Connectors" deviceset="CONN_10" device="NO_SILK_PTH_FEMALE"/>
 <part name="J2" library="SparkFun-Connectors" deviceset="CONN_10" device="NO_SILK_PTH_FEMALE"/>
+<part name="J3" library="SparkFun-Connectors" deviceset="BINDING_POST" device=""/>
+<part name="J4" library="SparkFun-Connectors" deviceset="BINDING_POST" device=""/>
+<part name="J5" library="SparkFun-Connectors" deviceset="BINDING_POST" device=""/>
+<part name="J6" library="SparkFun-Connectors" deviceset="BINDING_POST" device=""/>
+<part name="J7" library="SparkFun-Connectors" deviceset="BINDING_POST" device=""/>
+<part name="J8" library="SparkFun-Connectors" deviceset="BINDING_POST" device=""/>
 </parts>
 <sheets>
@@
 <attribute name="VALUE" x="-81.28" y="45.466" size="1.778" layer="96" align="top-center"/>
 </instance>
-<instance part="J37" gate="G$1" x="-312.42" y="287.02" smashed="yes">
-<attribute name="NAME" x="-313.436" y="288.798" size="1.778" layer="95" font="vector"/>
-<attribute name="VALUE" x="-313.436" y="283.972" size="1.778" layer="96" font="vector"/>
-</instance>
-<instance part="J38" gate="G$1" x="-312.42" y="281.94" smashed="yes">
-<attribute name="NAME" x="-313.436" y="283.718" size="1.778" layer="95" font="vector"/>
-<attribute name="VALUE" x="-313.436" y="278.892" size="1.778" layer="96" font="vector"/>
-</instance>
-<instance part="J39" gate="G$1" x="-215.9" y="180.34" smashed="yes" rot="R90">
-<attribute name="NAME" x="-217.678" y="179.324" size="1.778" layer="95" font="vector" rot="R90"/>
-<attribute name="VALUE" x="-212.852" y="179.324" size="1.778" layer="96" font="vector" rot="R90"/>
-</instance>
-<instance part="J40" gate="G$1" x="45.72" y="182.88" smashed="yes" rot="R90">
-<attribute name="NAME" x="43.942" y="181.864" size="1.778" layer="95" font="vector" rot="R90"/>
-<attribute name="VALUE" x="48.768" y="181.864" size="1.778" layer="96" font="vector" rot="R90"/>
-</instance>
-<instance part="J41" gate="G$1" x="-223.52" y="63.5" smashed="yes" rot="R90">
-<attribute name="NAME" x="-225.298" y="62.484" size="1.778" layer="95" font="vector" rot="R90"/>
-<attribute name="VALUE" x="-220.472" y="62.484" size="1.778" layer="96" font="vector" rot="R90"/>
-</instance>
-<instance part="J42" gate="G$1" x="50.8" y="63.5" smashed="yes" rot="R90">
-<attribute name="NAME" x="49.022" y="62.484" size="1.778" layer="95" font="vector" rot="R90"/>
-<attribute name="VALUE" x="53.848" y="62.484" size="1.778" layer="96" font="vector" rot="R90"/>
-</instance>
 <instance part="GND3" gate="1" x="-317.5" y="274.32" smashed="yes">
 <attribute name="VALUE" x="-317.5" y="274.066" size="1.778" layer="96" align="top-center"/>
@@
 <attribute name="VALUE" x="76.2" y="68.834" size="1.778" layer="96" font="vector"/>
 <attribute name="NAME" x="73.66" y="102.108" size="1.778" layer="95" font="vector"/>
+</instance>
+<instance part="J3" gate="G$1" x="-312.42" y="287.02" smashed="yes">
+<attribute name="NAME" x="-314.96" y="289.56" size="1.778" layer="95" font="vector"/>
+<attribute name="VALUE" x="-314.96" y="284.48" size="1.778" layer="95" font="vector" align="top-left"/>
+</instance>
+<instance part="J4" gate="G$1" x="-312.42" y="281.94" smashed="yes">
+<attribute name="NAME" x="-314.96" y="284.48" size="1.778" layer="95" font="vector"/>
+<attribute name="VALUE" x="-314.96" y="279.4" size="1.778" layer="95" font="vector" align="top-left"/>
+</instance>
+<instance part="J5" gate="G$1" x="-215.9" y="180.34" smashed="yes" rot="R90">
+<attribute name="NAME" x="-218.44" y="177.8" size="1.778" layer="95" font="vector" rot="R90"/>
+<attribute name="VALUE" x="-213.36" y="177.8" size="1.778" layer="95" font="vector" rot="R90" align="top-left"/>
+</instance>
+<instance part="J6" gate="G$1" x="50.8" y="180.34" smashed="yes" rot="R90">
+<attribute name="NAME" x="48.26" y="177.8" size="1.778" layer="95" font="vector" rot="R90"/>
+<attribute name="VALUE" x="53.34" y="177.8" size="1.778" layer="95" font="vector" rot="R90" align="top-left"/>
+</instance>
+<instance part="J7" gate="G$1" x="50.8" y="63.5" smashed="yes" rot="R90">
+<attribute name="NAME" x="48.26" y="60.96" size="1.778" layer="95" font="vector" rot="R90"/>
+<attribute name="VALUE" x="53.34" y="60.96" size="1.778" layer="95" font="vector" rot="R90" align="top-left"/>
+</instance>
+<instance part="J8" gate="G$1" x="-218.44" y="63.5" smashed="yes" rot="R90">
+<attribute name="NAME" x="-220.98" y="60.96" size="1.778" layer="95" font="vector" rot="R90"/>
+<attribute name="VALUE" x="-215.9" y="60.96" size="1.778" layer="95" font="vector" rot="R90" align="top-left"/>
 </instance>
 </instances>
@@
 </segment>
 <segment>
-<pinref part="J38" gate="G$1" pin="1"/>
+<wire x1="-317.5" y1="287.02" x2="-317.5" y2="281.94" width="0.1524" layer="91"/>
+<pinref part="GND3" gate="1" pin="GND"/>
+<pinref part="J3" gate="G$1" pin="P$1"/>
+<wire x1="-317.5" y1="281.94" x2="-317.5" y2="276.86" width="0.1524" layer="91"/>
+<wire x1="-317.5" y1="287.02" x2="-314.96" y2="287.02" width="0.1524" layer="91"/>
+<pinref part="J4" gate="G$1" pin="P$1"/>
 <wire x1="-314.96" y1="281.94" x2="-317.5" y2="281.94" width="0.1524" layer="91"/>
-<wire x1="-317.5" y1="281.94" x2="-317.5" y2="287.02" width="0.1524" layer="91"/>
-<pinref part="J37" gate="G$1" pin="1"/>
-<wire x1="-317.5" y1="287.02" x2="-314.96" y2="287.02" width="0.1524" layer="91"/>
 <junction x="-317.5" y="281.94"/>
-<wire x1="-317.5" y1="281.94" x2="-317.5" y2="276.86" width="0.1524" layer="91"/>
-<pinref part="GND3" gate="1" pin="GND"/>
 </segment>
 </net>
@@
 <junction x="-218.44" y="175.26"/>
 <wire x1="-218.44" y1="175.26" x2="-215.9" y2="175.26" width="0.1524" layer="91"/>
-<junction x="-215.9" y="175.26"/>
 <wire x1="-226.06" y1="175.26" x2="-223.52" y2="175.26" width="0.1524" layer="91"/>
 <junction x="-226.06" y="175.26"/>
@@
 <wire x1="-223.52" y1="175.26" x2="-220.98" y2="175.26" width="0.1524" layer="91"/>
 <junction x="-223.52" y="175.26"/>
-<pinref part="J39" gate="G$1" pin="1"/>
-<wire x1="-215.9" y1="177.8" x2="-215.9" y2="175.26" width="0.1524" layer="91"/>
+<pinref part="J5" gate="G$1" pin="P$1"/>
+<wire x1="-215.9" y1="175.26" x2="-215.9" y2="177.8" width="0.1524" layer="91"/>
+<junction x="-215.9" y="175.26"/>
 </segment>
 </net>
 <net name="N$2" class="0">
 <segment>
-<wire x1="45.72" y1="175.26" x2="45.72" y2="180.34" width="0.1524" layer="91"/>
-<pinref part="J40" gate="G$1" pin="1"/>
 <pinref part="J45" gate="G$1" pin="3"/>
 <pinref part="J45" gate="G$1" pin="40"/>
@@
 <junction x="45.72" y="175.26"/>
 <junction x="50.8" y="175.26"/>
+<pinref part="J6" gate="G$1" pin="P$1"/>
+<wire x1="50.8" y1="175.26" x2="50.8" y2="177.8" width="0.1524" layer="91"/>
 </segment>
 </net>
@@
 <wire x1="45.72" y1="58.42" x2="48.26" y2="58.42" width="0.1524" layer="91"/>
 <wire x1="48.26" y1="58.42" x2="50.8" y2="58.42" width="0.1524" layer="91"/>
-<wire x1="50.8" y1="58.42" x2="50.8" y2="60.96" width="0.1524" layer="91"/>
-<pinref part="J42" gate="G$1" pin="1"/>
 <pinref part="J46" gate="G$1" pin="1"/>
-<junction x="50.8" y="58.42"/>
 <pinref part="J46" gate="G$1" pin="2"/>
 <junction x="48.26" y="58.42"/>
@@
 <pinref part="J46" gate="G$1" pin="40"/>
 <junction x="-48.26" y="58.42"/>
+<pinref part="J7" gate="G$1" pin="P$1"/>
+<wire x1="50.8" y1="58.42" x2="50.8" y2="60.96" width="0.1524" layer="91"/>
+<junction x="50.8" y="58.42"/>
 </segment>
 </net>
@@
 <wire x1="-228.6" y1="58.42" x2="-226.06" y2="58.42" width="0.1524" layer="91"/>
 <wire x1="-226.06" y1="58.42" x2="-223.52" y2="58.42" width="0.1524" layer="91"/>
-<wire x1="-223.52" y1="58.42" x2="-223.52" y2="60.96" width="0.1524" layer="91"/>
-<pinref part="J41" gate="G$1" pin="1"/>
 <wire x1="-223.52" y1="58.42" x2="-220.98" y2="58.42" width="0.1524" layer="91"/>
 <junction x="-223.52" y="58.42"/>
@@
 <junction x="-314.96" y="58.42"/>
 <pinref part="J48" gate="G$1" pin="40"/>
-</segment>
-</net>
+<pinref part="J8" gate="G$1" pin="P$1"/>
+<wire x1="-218.44" y1="58.42" x2="-218.44" y2="60.96" width="0.1524" layer="91"/>
+<junction x="-218.44" y="58.42"/>
+</segment>
+</net>
